File: flame-detect-pcb.kicad_pcb (KiCad board)
At the start: 2 copper layers, 82.5 x 101.6 mm, 57 parts, among them IC1 ATMEGA328-P, IC2 CH340G, P0 RELAY_(JSM1A-12V-4), P1 RELAY_(JSM1A-12V-4), P2 RELAY_(JSM1A-12V-4), P3 RELAY_(JSM1A-12V-4), P4 RELAY_(JSM1A-12V-4), P5 RELAY_(JSM1A-12V-4), Q1 Q_NPN_BEC, Q12 Q_NPN, Q13 Q_NPN, Q14 Q_NPN, Q15 Q_NPN, Q16 Q_NPN, Q17 Q_NPN, Q4 Q_NPN_BEC, Q5 Q_NPN_BEC, Q6 Q_NPN_BEC, Q7 Q_NPN_BEC, Q8 Q_NPN_BEC, Q9 Q_NPN_BEC, U1 NCV7805BDTRKG, X1 Crystal_GND2, X2 Crystal_GND2

Commit message: - Created transformer block and footprint.
Parts:
- C1, C2, D3, D4, D5, D6, D7, D8, R1, R10, R11, R12, R13, R14, R15, R16, R17, R18, R2, R21, R22, R23, R24, R25, R26, R27, R28, R7, R8, R9: footprint USBdio-PCB:R_1206_HandSoldering_(narrow) -> flame-detect-pcb:R_1206_HandSoldering_(narrow)
- CONN_1: footprint USBdio-PCB:DEUTSCH_CONN_(DTM13-12PA-12PB-R008) -> flame-detect-pcb:DEUTSCH_CONN_(DTM13-12PA-12PB-R008)
- D9: footprint USBdio-PCB:SCHOTTKY_(PMEG3030EP,115) -> flame-detect-pcb:SCHOTTKY_(PMEG3030EP,115)
- IC2: footprint USBdio-PCB:CH340G -> flame-detect-pcb:CH340G
- P0, P1, P2, P3, P4, P5: footprint USBdio-PCB:RELAY_(JSM1A-12V-4) -> flame-detect-pcb:RELAY_(JSM1A-12V-4)
- U1: footprint USBdio-PCB:REGULATOR_(NCV7805BDTRKG) -> flame-detect-pcb:REGULATOR_(NCV7805BDTRKG)
- X1, X2: footprint USBdio-PCB:RESONATOR_(CSTCE16M0V53C-R0) -> flame-detect-pcb:RESONATOR_(CSTCE16M0V53C-R0)
