File: CAN.sch (KiCad schematic (older format))
At the start: 13 parts, among them U7 MCP2515T-I/SO, U8 MCP2551-I/SN

Commit message: - Finished footprints.
Parts:
- CAN_HI_1, CAN_LO_1: footprint (none) -> flame-detect-pcb:KEYSTONE_SPADE_TERM_(1287)
- CAN_TERM_1: footprint (none) -> Pin_Headers:Pin_Header_Straight_1x02_Pitch2.54mm_SMD_Pin1Left
- U7: footprint (none) -> Housings_SOIC:SOIC-18W_7.5x11.6mm_Pitch1.27mm
- XTAL2: footprint (none) -> Crystals:Crystal_SMD_HC49-SD
Changed lines of the file:
@@
 F 0 "XTAL2" H 3350 4150 50  0000 C CNN
 F 1 "Crystal" H 3350 3850 50  0001 C CNN
-F 2 "" H 3350 4000 50  0001 C CNN
+F 2 "Crystals:Crystal_SMD_HC49-SD" H 3350 4000 50  0001 C CNN
 F 3 "" H 3350 4000 50  0001 C CNN
 	1    3350 4000
@@
 F 0 "U7" H 4100 4325 50  0000 R CNN
 F 1 "MCP2515T-I/SO" H 5250 4350 50  0000 R TNN
-F 2 "" H 4500 2650 50  0001 C CIN
+F 2 "Housings_SOIC:SOIC-18W_7.5x11.6mm_Pitch1.27mm" H 4500 2650 50  0001 C CIN
 F 3 "" H 4600 2750 50  0001 C CNN
 	1    4500 3550
@@
 F 0 "CAN_TERM_1" H 8700 3800 50  0000 C CNN
 F 1 "CONN_01X02" V 8800 3650 50  0001 C CNN
-F 2 "" H 8700 3650 50  0001 C CNN
+F 2 "Pin_Headers:Pin_Header_Straight_1x02_Pitch2.54mm_SMD_Pin1Left" H 8700 3650 50  0001 C CNN
 F 3 "" H 8700 3650 50  0001 C CNN
 	1    8700 3650
@@
 F 0 "CAN_HI_1" H 8700 3050 50  0000 C CNN
 F 1 "CONN_01X01" V 8800 2950 50  0001 C CNN
-F 2 "" H 8700 2950 50  0001 C CNN
+F 2 "flame-detect-pcb:KEYSTONE_SPADE_TERM_(1287)" H 8700 2950 50  0001 C CNN
 F 3 "" H 8700 2950 50  0001 C CNN
 	1    8700 2950
@@
 F 0 "CAN_LO_1" H 8700 3250 50  0000 C CNN
 F 1 "CONN_01X01" V 8800 3150 50  0001 C CNN
-F 2 "" H 8700 3150 50  0001 C CNN
+F 2 "flame-detect-pcb:KEYSTONE_SPADE_TERM_(1287)" H 8700 3150 50  0001 C CNN
 F 3 "" H 8700 3150 50  0001 C CNN
 	1    8700 3150

Commit message: - Finished PCB layout.
Parts:
- added CAN_HI_2, CAN_LO_2: CONN_01X01, flame-detect-pcb:KEYSTONE_SPADE_TERM_(1287), symbol CONN_01X01
Connections:
- net at CAN_LO_1.1 (P1), R5.1, U8.6 (CANL): now also CAN_LO_2.1 (P1)
- net at CAN_HI_1.1 (P1), CAN_TERM_1.1 (P1), U8.7 (CANH): now also CAN_HI_2.1 (P1)
Other:
- moved on the sheet: CAN_HI_1
Changed lines of the file:
@@
 $EndComp
 $Comp
-L GND #PWR013
+L GND #PWR014
 U 1 1 5AAF95EC
 P 2550 4550
-F 0 "#PWR013" H 2550 4300 50  0001 C CNN
+F 0 "#PWR014" H 2550 4300 50  0001 C CNN
 F 1 "GND" H 2550 4400 50  0000 C CNN
 F 2 "" H 2550 4550 50  0000 C CNN
@@
 NoConn ~ 3900 3950
 $Comp
-L GND #PWR014
+L GND #PWR015
 U 1 1 5AAF989F
 P 4500 4550
-F 0 "#PWR014" H 4500 4300 50  0001 C CNN
+F 0 "#PWR015" H 4500 4300 50  0001 C CNN
 F 1 "GND" H 4500 4400 50  0000 C CNN
 F 2 "" H 4500 4550 50  0000 C CNN
@@
 	1    0    0    -1
 $EndComp
-Wire Wire Line
-	3050 3750 3900 3750
-Wire Wire Line
-	3050 4250 3650 4250
-Wire Wire Line
-	3650 4250 3650 3850
-Wire Wire Line
-	3650 3850 3900 3850
-Wire Wire Line
-	3350 3850 3350 3750
-Connection ~ 3350 3750
-Wire Wire Line
-	3350 4150 3350 4250
-Connection ~ 3350 4250
-Wire Wire Line
-	2550 3750 2550 4550
-Wire Wire Line
-	2550 3750 2750 3750
-Wire Wire Line
-	2550 4250 2750 4250
-Connection ~ 2550 4250
-Wire Wire Line
-	4500 4350 4500 4550
 Text GLabel 2550 2050 0    60   Input ~ 0
 5V
-Wire Wire Line
-	2550 2050 7050 2050
-Wire Wire Line
-	5800 2050 4500 2050
-Wire Wire Line
-	4500 2050 4500 2750
 $Comp
 L C C11
@@
 	-1   0    0    1
 $EndComp
-Wire Wire Line
-	3450 2150 3450 2050
-Connection ~ 3450 2050
-Wire Wire Line
-	6250 2150 6250 2050
-Connection ~ 6250 2050
-$Comp
-L GND #PWR015
+$Comp
+L GND #PWR016
 U 1 1 5AAF9AF5
 P 3450 2550
-F 0 "#PWR015" H 3450 2300 50  0001 C CNN
+F 0 "#PWR016" H 3450 2300 50  0001 C CNN
 F 1 "GND" H 3450 2400 50  0000 C CNN
 F 2 "" H 3450 2550 50  0000 C CNN
@@
 $EndComp
 $Comp
-L GND #PWR016
+L GND #PWR017
 U 1 1 5AAF9B15
 P 6250 2550
-F 0 "#PWR016" H 6250 2300 50  0001 C CNN
+F 0 "#PWR017" H 6250 2300 50  0001 C CNN
 F 1 "GND" H 6250 2400 50  0000 C CNN
 F 2 "" H 6250 2550 50  0000 C CNN
@@
 	1    0    0    -1
 $EndComp
-Wire Wire Line
-	3450 2450 3450 2550
-Wire Wire Line
-	6250 2450 6250 2550
 $Comp
 L R R3
@@
 	0    1    1    0
 $EndComp
-Wire Wire Line
-	5100 4150 5300 4150
-Wire Wire Line
-	5600 4150 5800 4150
-Wire Wire Line
-	5800 4150 5800 2050
-Connection ~ 4500 2050
-Wire Wire Line
-	5100 2950 6550 2950
-Wire Wire Line
-	5100 3050 6350 3050
-Wire Wire Line
-	6350 3050 6350 2850
-Wire Wire Line
-	6350 2850 6550 2850
-Wire Wire Line
-	7050 2050 7050 2650
-Connection ~ 5800 2050
-$Comp
-L GND #PWR017
+$Comp
+L GND #PWR018
 U 1 1 5AAF9DE1
 P 7050 4550
-F 0 "#PWR017" H 7050 4300 50  0001 C CNN
+F 0 "#PWR018" H 7050 4300 50  0001 C CNN
 F 1 "GND" H 7050 4400 50  0000 C CNN
 F 2 "" H 7050 4550 50  0000 C CNN
@@
 	1    0    0    -1
 $EndComp
-Wire Wire Line
-	7050 3450 7050 4550
 NoConn ~ 6550 3150
 $Comp
@@
 	1    0    0    1
 $EndComp
-Wire Wire Line
-	6350 3250 6350 3600
-Wire Wire Line
-	6350 3250 6550 3250
-$Comp
-L GND #PWR018
+$Comp
+L GND #PWR019
 U 1 1 5AAF9F1C
 P 6350 4550
-F 0 "#PWR018" H 6350 4300 50  0001 C CNN
+F 0 "#PWR019" H 6350 4300 50  0001 C CNN
 F 1 "GND" H 6350 4400 50  0000 C CNN
 F 2 "" H 6350 4550 50  0000 C CNN
@@
 	1    0    0    -1
 $EndComp
-Wire Wire Line
-	6350 3900 6350 4550
 Text GLabel 2550 2950 0    60   Input ~ 0
 MOSI
-Wire Wire Line
-	2550 2950 3900 2950
 Text GLabel 2550 3050 0    60   Input ~ 0
 MISO
@@
 Text GLabel 2550 3250 0    60   Input ~ 0
 SCK
-Wire Wire Line
-	2550 3050 3900 3050
-Wire Wire Line
-	3900 3150 2550 3150
-Wire Wire Line
-	2550 3250 3900 3250
 Text GLabel 5350 3550 2    60   Input ~ 0
 INT
-Wire Wire Line
-	5100 3550 5350 3550
 NoConn ~ 5100 3850
 NoConn ~ 5100 3950
@@
 L CONN_01X01 CAN_HI_1
 U 1 1 5AAFAD8C
-P 8700 2950
-F 0 "CAN_HI_1" H 8700 3050 50  0000 C CNN
-F 1 "CONN_01X01" V 8800 2950 50  0001 C CNN
-F 2 "flame-detect-pcb:KEYSTONE_SPADE_TERM_(1287)" H 8700 2950 50  0001 C CNN
-F 3 "" H 8700 2950 50  0001 C CNN
-	1    8700 2950
+P 8700 2750
+F 0 "CAN_HI_1" H 8700 2850 50  0000 C CNN
+F 1 "CONN_01X01" V 8800 2750 50  0001 C CNN
+F 2 "flame-detect-pcb:KEYSTONE_SPADE_TERM_(1287)" H 8700 2750 50  0001 C CNN
+F 3 "" H 8700 2750 50  0001 C CNN
+	1    8700 2750
 	1    0    0    -1
 $EndComp
@@
 	1    0    0    -1
 $EndComp
-Wire Wire Line
-	7550 2950 8500 2950
-Wire Wire Line
-	7550 3150 8500 3150
-Wire Wire Line
-	8500 3600 8350 3600
-Wire Wire Line
-	8350 3600 8350 2950
-Connection ~ 8350 2950
 $Comp
 L R R5
@@
 	0    -1   1    0
 $EndComp
+$Comp
+L CONN_01X01 CAN_HI_2
+U 1 1 5AB19FCB
+P 8700 2950
+F 0 "CAN_HI_2" H 8700 3050 50  0000 C CNN
+F 1 "CONN_01X01" V 8800 2950 50  0001 C CNN
+F 2 "flame-detect-pcb:KEYSTONE_SPADE_TERM_(1287)" H 8700 2950 50  0001 C CNN
+F 3 "" H 8700 2950 50  0001 C CNN
+	1    8700 2950
+	1    0    0    -1
+$EndComp
+$Comp
+L CONN_01X01 CAN_LO_2
+U 1 1 5AB1A123
+P 8700 3350
+F 0 "CAN_LO_2" H 8700 3450 50  0000 C CNN
+F 1 "CONN_01X01" V 8800 3350 50  0001 C CNN
+F 2 "flame-detect-pcb:KEYSTONE_SPADE_TERM_(1287)" H 8700 3350 50  0001 C CNN
+F 3 "" H 8700 3350 50  0001 C CNN
+	1    8700 3350
+	1    0    0    -1
+$EndComp
+Wire Wire Line
+	3050 3750 3900 3750
+Wire Wire Line
+	3050 4250 3650 4250
+Wire Wire Line
+	3650 4250 3650 3850
+Wire Wire Line
+	3650 3850 3900 3850
+Wire Wire Line
+	3350 3850 3350 3750
+Connection ~ 3350 3750
+Wire Wire Line
+	3350 4150 3350 4250
+Connection ~ 3350 4250
+Wire Wire Line
+	2550 3750 2550 4550
+Wire Wire Line
+	2550 3750 2750 3750
+Wire Wire Line
+	2550 4250 2750 4250
+Connection ~ 2550 4250
+Wire Wire Line
+	4500 4350 4500 4550
+Wire Wire Line
+	2550 2050 7050 2050
+Wire Wire Line
+	5800 2050 4500 2050
+Wire Wire Line
+	4500 2050 4500 2750
+Wire Wire Line
+	3450 2150 3450 2050
+Connection ~ 3450 2050
+Wire Wire Line
+	6250 2150 6250 2050
+Connection ~ 6250 2050
+Wire Wire Line
+	3450 2450 3450 2550
+Wire Wire Line
+	6250 2450 6250 2550
+Wire Wire Line
+	5100 4150 5300 4150
+Wire Wire Line
+	5600 4150 5800 4150
+Wire Wire Line
+	5800 4150 5800 2050
+Connection ~ 4500 2050
+Wire Wire Line
+	5100 2950 6550 2950
+Wire Wire Line
+	5100 3050 6350 3050
+Wire Wire Line
+	6350 3050 6350 2850
+Wire Wire Line
+	6350 2850 6550 2850
+Wire Wire Line
+	7050 2050 7050 2650
+Connection ~ 5800 2050
+Wire Wire Line
+	7050 3450 7050 4550
+Wire Wire Line
+	6350 3250 6350 3600
+Wire Wire Line
+	6350 3250 6550 3250
+Wire Wire Line
+	6350 3900 6350 4550
+Wire Wire Line
+	2550 2950 3900 2950
+Wire Wire Line
+	2550 3050 3900 3050
+Wire Wire Line
+	3900 3150 2550 3150
+Wire Wire Line
+	2550 3250 3900 3250
+Wire Wire Line
+	5100 3550 5350 3550
+Wire Wire Line
+	7550 2950 8500 2950
+Wire Wire Line
+	7550 3150 8500 3150
+Wire Wire Line
+	8350 3600 8500 3600
+Wire Wire Line
+	8350 2750 8350 3600
+Connection ~ 8350 2950
 Wire Wire Line
 	8500 3700 8250 3700
@@
 	7750 3700 7750 3150
 Connection ~ 7750 3150
+Wire Wire Line
+	8500 2750 8350 2750
+Wire Wire Line
+	8500 3350 8450 3350
+Wire Wire Line
+	8450 3350 8450 3150
+Connection ~ 8450 3150
 $EndSCHEMATC

Commit message: - Fixed several bugs.
Parts:
- CAN_TERM_1: footprint Pin_Headers:Pin_Header_Straight_1x02_Pitch2.54mm_SMD_Pin1Left -> Pin_Headers:Pin_Header_Straight_1x02_Pitch2.54mm_SMD_Pin1Right
Changed lines of the file:
@@
 $EndComp
 $Comp
-L GND #PWR014
+L GND #PWR015
 U 1 1 5AAF95EC
 P 2550 4550
-F 0 "#PWR014" H 2550 4300 50  0001 C CNN
+F 0 "#PWR015" H 2550 4300 50  0001 C CNN
 F 1 "GND" H 2550 4400 50  0000 C CNN
 F 2 "" H 2550 4550 50  0000 C CNN
@@
 NoConn ~ 3900 3950
 $Comp
-L GND #PWR015
+L GND #PWR016
 U 1 1 5AAF989F
 P 4500 4550
-F 0 "#PWR015" H 4500 4300 50  0001 C CNN
+F 0 "#PWR016" H 4500 4300 50  0001 C CNN
 F 1 "GND" H 4500 4400 50  0000 C CNN
 F 2 "" H 4500 4550 50  0000 C CNN
@@
 $EndComp
 $Comp
-L GND #PWR016
+L GND #PWR017
 U 1 1 5AAF9AF5
 P 3450 2550
-F 0 "#PWR016" H 3450 2300 50  0001 C CNN
+F 0 "#PWR017" H 3450 2300 50  0001 C CNN
 F 1 "GND" H 3450 2400 50  0000 C CNN
 F 2 "" H 3450 2550 50  0000 C CNN
@@
 $EndComp
 $Comp
-L GND #PWR017
+L GND #PWR018
 U 1 1 5AAF9B15
 P 6250 2550
-F 0 "#PWR017" H 6250 2300 50  0001 C CNN
+F 0 "#PWR018" H 6250 2300 50  0001 C CNN
 F 1 "GND" H 6250 2400 50  0000 C CNN
 F 2 "" H 6250 2550 50  0000 C CNN
@@
 $EndComp
 $Comp
-L GND #PWR018
+L GND #PWR019
 U 1 1 5AAF9DE1
 P 7050 4550
-F 0 "#PWR018" H 7050 4300 50  0001 C CNN
+F 0 "#PWR019" H 7050 4300 50  0001 C CNN
 F 1 "GND" H 7050 4400 50  0000 C CNN
 F 2 "" H 7050 4550 50  0000 C CNN
@@
 $EndComp
 $Comp
-L GND #PWR019
+L GND #PWR020
 U 1 1 5AAF9F1C
 P 6350 4550
-F 0 "#PWR019" H 6350 4300 50  0001 C CNN
+F 0 "#PWR020" H 6350 4300 50  0001 C CNN
 F 1 "GND" H 6350 4400 50  0000 C CNN
 F 2 "" H 6350 4550 50  0000 C CNN
@@
 F 0 "CAN_TERM_1" H 8700 3800 50  0000 C CNN
 F 1 "CONN_01X02" V 8800 3650 50  0001 C CNN
-F 2 "Pin_Headers:Pin_Header_Straight_1x02_Pitch2.54mm_SMD_Pin1Left" H 8700 3650 50  0001 C CNN
+F 2 "Pin_Headers:Pin_Header_Straight_1x02_Pitch2.54mm_SMD_Pin1Right" H 8700 3650 50  0001 C CNN
 F 3 "" H 8700 3650 50  0001 C CNN
 	1    8700 3650
