File: FLAME_DETECT_1-4.sch (KiCad schematic (older format))
At the start: 58 parts, among them Q1 MMBT2907, Q2 MMBT2907, Q3 MMBT2907, Q4 MMBT2907, U1 LM358, U2 LM358

Commit message: - Finished footprints.
Parts:
- D10, D11, D12, D2, D3, D4, D5, D8: footprint Diodes_SMD:D_0805 -> Diodes_SMD:D_SOD-123
- D13, D14, D6, D7: footprint (none) -> LEDs:LED_1206
- FLAME_1, FLAME_2, FLAME_3, FLAME_4: footprint (none) -> flame-detect-pcb:KEYSTONE_SPADE_TERM_(1287)
- U1, U2: footprint (none) -> Housings_SOIC:SOIC-8_3.9x4.9mm_Pitch1.27mm
Changed lines of the file:
@@
 F 0 "FLAME_1" H 4950 1600 50  0000 C CNN
 F 1 "CONN_01X01" V 5050 1500 50  0001 C CNN
-F 2 "" H 4950 1500 50  0001 C CNN
+F 2 "flame-detect-pcb:KEYSTONE_SPADE_TERM_(1287)" H 4950 1500 50  0001 C CNN
 F 3 "" H 4950 1500 50  0001 C CNN
 	1    4950 1500
@@
 F 0 "D2" H 1700 2000 50  0000 C CNN
 F 1 "BAV21W-7-F" H 1700 1800 50  0000 C CNN
-F 2 "Diodes_SMD:D_0805" H 1700 1900 50  0001 C CNN
+F 2 "Diodes_SMD:D_SOD-123" H 1700 1900 50  0001 C CNN
 F 3 "" H 1700 1900 50  0001 C CNN
 	1    1700 1900
@@
 F 0 "U1" H 3500 2500 50  0000 L CNN
 F 1 "LM358" H 3500 2100 50  0000 L CNN
-F 2 "" H 3500 2300 50  0001 C CNN
+F 2 "Housings_SOIC:SOIC-8_3.9x4.9mm_Pitch1.27mm" H 3500 2300 50  0001 C CNN
 F 3 "" H 3500 2300 50  0001 C CNN
 	1    3500 2300
@@
 F 0 "U1" H 3500 5250 50  0000 L CNN
 F 1 "LM358" H 3500 4850 50  0000 L CNN
-F 2 "" H 3500 5050 50  0001 C CNN
+F 2 "Housings_SOIC:SOIC-8_3.9x4.9mm_Pitch1.27mm" H 3500 5050 50  0001 C CNN
 F 3 "" H 3500 5050 50  0001 C CNN
 	2    3500 5050
@@
 F 0 "D4" H 4050 2900 50  0000 C CNN
 F 1 "BZT52C5V1-TP" H 4050 2700 50  0000 C CNN
-F 2 "Diodes_SMD:D_0805" H 4050 2800 50  0001 C CNN
+F 2 "Diodes_SMD:D_SOD-123" H 4050 2800 50  0001 C CNN
 F 3 "" H 4050 2800 50  0001 C CNN
 	1    4050 2800
@@
 F 0 "D6" H 4450 3000 50  0000 C CNN
 F 1 "LED" H 4450 2800 50  0000 C CNN
-F 2 "" H 4450 2900 50  0001 C CNN
+F 2 "LEDs:LED_1206" H 4450 2900 50  0001 C CNN
 F 3 "" H 4450 2900 50  0001 C CNN
 	1    4450 2900
@@
 F 0 "FLAME_2" H 4950 4350 50  0000 C CNN
 F 1 "CONN_01X01" V 5050 4250 50  0001 C CNN
-F 2 "" H 4950 4250 50  0001 C CNN
+F 2 "flame-detect-pcb:KEYSTONE_SPADE_TERM_(1287)" H 4950 4250 50  0001 C CNN
 F 3 "" H 4950 4250 50  0001 C CNN
 	1    4950 4250
@@
 F 0 "D3" H 1700 4750 50  0000 C CNN
 F 1 "BAV21W-7-F" H 1700 4550 50  0000 C CNN
-F 2 "Diodes_SMD:D_0805" H 1700 4650 50  0001 C CNN
+F 2 "Diodes_SMD:D_SOD-123" H 1700 4650 50  0001 C CNN
 F 3 "" H 1700 4650 50  0001 C CNN
 	1    1700 4650
@@
 F 0 "D5" H 4050 5650 50  0000 C CNN
 F 1 "BZT52C5V1-TP" H 4050 5450 50  0000 C CNN
-F 2 "Diodes_SMD:D_0805" H 4050 5550 50  0001 C CNN
+F 2 "Diodes_SMD:D_SOD-123" H 4050 5550 50  0001 C CNN
 F 3 "" H 4050 5550 50  0001 C CNN
 	1    4050 5550
@@
 F 0 "D7" H 4450 5750 50  0000 C CNN
 F 1 "LED" H 4450 5550 50  0000 C CNN
-F 2 "" H 4450 5650 50  0001 C CNN
+F 2 "LEDs:LED_1206" H 4450 5650 50  0001 C CNN
 F 3 "" H 4450 5650 50  0001 C CNN
 	1    4450 5650
@@
 F 0 "FLAME_3" H 10100 1600 50  0000 C CNN
 F 1 "CONN_01X01" V 10200 1500 50  0001 C CNN
-F 2 "" H 10100 1500 50  0001 C CNN
+F 2 "flame-detect-pcb:KEYSTONE_SPADE_TERM_(1287)" H 10100 1500 50  0001 C CNN
 F 3 "" H 10100 1500 50  0001 C CNN
 	1    10100 1500
@@
 F 0 "D8" H 6850 2000 50  0000 C CNN
 F 1 "BAV21W-7-F" H 6850 1800 50  0000 C CNN
-F 2 "Diodes_SMD:D_0805" H 6850 1900 50  0001 C CNN
+F 2 "Diodes_SMD:D_SOD-123" H 6850 1900 50  0001 C CNN
 F 3 "" H 6850 1900 50  0001 C CNN
 	1    6850 1900
@@
 F 0 "U2" H 8650 2500 50  0000 L CNN
 F 1 "LM358" H 8650 2100 50  0000 L CNN
-F 2 "" H 8650 2300 50  0001 C CNN
+F 2 "Housings_SOIC:SOIC-8_3.9x4.9mm_Pitch1.27mm" H 8650 2300 50  0001 C CNN
 F 3 "" H 8650 2300 50  0001 C CNN
 	1    8650 2300
@@
 F 0 "D11" H 9200 2900 50  0000 C CNN
 F 1 "BZT52C5V1-TP" H 9200 2700 50  0000 C CNN
-F 2 "Diodes_SMD:D_0805" H 9200 2800 50  0001 C CNN
+F 2 "Diodes_SMD:D_SOD-123" H 9200 2800 50  0001 C CNN
 F 3 "" H 9200 2800 50  0001 C CNN
 	1    9200 2800
@@
 F 0 "D13" H 9600 3000 50  0000 C CNN
 F 1 "LED" H 9600 2800 50  0000 C CNN
-F 2 "" H 9600 2900 50  0001 C CNN
+F 2 "LEDs:LED_1206" H 9600 2900 50  0001 C CNN
 F 3 "" H 9600 2900 50  0001 C CNN
 	1    9600 2900
@@
 F 0 "FLAME_4" H 10100 4350 50  0000 C CNN
 F 1 "CONN_01X01" V 10200 4250 50  0001 C CNN
-F 2 "" H 10100 4250 50  0001 C CNN
+F 2 "flame-detect-pcb:KEYSTONE_SPADE_TERM_(1287)" H 10100 4250 50  0001 C CNN
 F 3 "" H 10100 4250 50  0001 C CNN
 	1    10100 4250
@@
 F 0 "D10" H 6850 4750 50  0000 C CNN
 F 1 "BAV21W-7-F" H 6850 4550 50  0000 C CNN
-F 2 "Diodes_SMD:D_0805" H 6850 4650 50  0001 C CNN
+F 2 "Diodes_SMD:D_SOD-123" H 6850 4650 50  0001 C CNN
 F 3 "" H 6850 4650 50  0001 C CNN
 	1    6850 4650
@@
 F 0 "D12" H 9200 5650 50  0000 C CNN
 F 1 "BZT52C5V1-TP" H 9200 5450 50  0000 C CNN
-F 2 "Diodes_SMD:D_0805" H 9200 5550 50  0001 C CNN
+F 2 "Diodes_SMD:D_SOD-123" H 9200 5550 50  0001 C CNN
 F 3 "" H 9200 5550 50  0001 C CNN
 	1    9200 5550
@@
 F 0 "D14" H 9600 5750 50  0000 C CNN
 F 1 "LED" H 9600 5550 50  0000 C CNN
-F 2 "" H 9600 5650 50  0001 C CNN
+F 2 "LEDs:LED_1206" H 9600 5650 50  0001 C CNN
 F 3 "" H 9600 5650 50  0001 C CNN
 	1    9600 5650
@@
 F 0 "U2" H 8650 5250 50  0000 L CNN
 F 1 "LM358" H 8650 4850 50  0000 L CNN
-F 2 "" H 8650 5050 50  0001 C CNN
+F 2 "Housings_SOIC:SOIC-8_3.9x4.9mm_Pitch1.27mm" H 8650 5050 50  0001 C CNN
 F 3 "" H 8650 5050 50  0001 C CNN
 	2    8650 5050

Commit message: - Fixed several bugs.
Parts:
- R18, R19, R35, R36: value 1M -> 10K
Connections:
- net at Q1.3 (C): now also D2.2 (A); no longer D2.1 (K)
- net at C12.1, R8.1, U1.3 (+): now also D2.1 (K); no longer D2.2 (A)
- net at C13.1, R9.1, U1.5 (+): now also D3.1 (K); no longer D3.2 (A)
- net at Q2.3 (C): now also D3.2 (A); no longer D3.1 (K)
- net at Q3.3 (C): now also D8.2 (A); no longer D8.1 (K)
- net at C16.1, R24.1, U2.3 (+): now also D8.1 (K); no longer D8.2 (A)
- net at Q4.3 (C): now also D10.2 (A); no longer D10.1 (K)
- net at C17.1, R25.1, U2.5 (+): now also D10.1 (K); no longer D10.2 (A)
Changed lines of the file:
@@
 F 3 "" H 1700 1900 50  0001 C CNN
 	1    1700 1900
-	0    1    1    0
+	0    -1   -1   0
 $EndComp
 Wire Wire Line
@@
 	1700 2050 1700 2650
 $Comp
-L GND #PWR020
+L GND #PWR021
 U 1 1 5AAF0F0F
 P 1700 3100
-F 0 "#PWR020" H 1700 2850 50  0001 C CNN
+F 0 "#PWR021" H 1700 2850 50  0001 C CNN
 F 1 "GND" H 1700 2950 50  0000 C CNN
 F 2 "" H 1700 3100 50  0001 C CNN
@@
 Connection ~ 1700 2400
 $Comp
-L GND #PWR021
+L GND #PWR022
 U 1 1 5AAF12ED
 P 2150 3100
-F 0 "#PWR021" H 2150 2850 50  0001 C CNN
+F 0 "#PWR022" H 2150 2850 50  0001 C CNN
 F 1 "GND" H 2150 2950 50  0000 C CNN
 F 2 "" H 2150 3100 50  0001 C CNN
@@
 P 3700 1850
 F 0 "R18" V 3780 1850 50  0000 C CNN
-F 1 "1M" V 3600 1850 50  0000 C CNN
+F 1 "10K" V 3600 1850 50  0000 C CNN
 F 2 "Resistors_SMD:R_0805" V 3630 1850 50  0001 C CNN
 F 3 "" H 3700 1850 50  0001 C CNN
@@
 $EndComp
 $Comp
-L GND #PWR022
+L GND #PWR023
 U 1 1 5AAF18A4
 P 3000 2000
-F 0 "#PWR022" H 3000 1750 50  0001 C CNN
+F 0 "#PWR023" H 3000 1750 50  0001 C CNN
 F 1 "GND" H 3000 1850 50  0000 C CNN
 F 2 "" H 3000 2000 50  0001 C CNN
@@
 Connection ~ 4050 2300
 $Comp
-L GND #PWR023
+L GND #PWR024
 U 1 1 5AAF1AA4
 P 4050 3100
-F 0 "#PWR023" H 4050 2850 50  0001 C CNN
+F 0 "#PWR024" H 4050 2850 50  0001 C CNN
 F 1 "GND" H 4050 2950 50  0000 C CNN
 F 2 "" H 4050 3100 50  0001 C CNN
@@
 Connection ~ 4450 2300
 $Comp
-L GND #PWR024
+L GND #PWR025
 U 1 1 5AAF1E49
 P 4450 3100
-F 0 "#PWR024" H 4450 2850 50  0001 C CNN
+F 0 "#PWR025" H 4450 2850 50  0001 C CNN
 F 1 "GND" H 4450 2950 50  0000 C CNN
 F 2 "" H 4450 3100 50  0001 C CNN
@@
 F 3 "" H 1700 4650 50  0001 C CNN
 	1    1700 4650
-	0    1    1    0
+	0    -1   -1   0
 $EndComp
 Wire Wire Line
@@
 	1700 4800 1700 5400
 $Comp
-L GND #PWR025
+L GND #PWR026
 U 1 1 5AAF3C27
 P 1700 5850
-F 0 "#PWR025" H 1700 5600 50  0001 C CNN
+F 0 "#PWR026" H 1700 5600 50  0001 C CNN
 F 1 "GND" H 1700 5700 50  0000 C CNN
 F 2 "" H 1700 5850 50  0001 C CNN
@@
 Connection ~ 1700 5150
 $Comp
-L GND #PWR026
+L GND #PWR027
 U 1 1 5AAF3C38
 P 2150 5850
-F 0 "#PWR026" H 2150 5600 50  0001 C CNN
+F 0 "#PWR027" H 2150 5600 50  0001 C CNN
 F 1 "GND" H 2150 5700 50  0000 C CNN
 F 2 "" H 2150 5850 50  0001 C CNN
@@
 P 3700 4600
 F 0 "R19" V 3780 4600 50  0000 C CNN
-F 1 "1M" V 3600 4600 50  0000 C CNN
+F 1 "10K" V 3600 4600 50  0000 C CNN
 F 2 "Resistors_SMD:R_0805" V 3630 4600 50  0001 C CNN
 F 3 "" H 3700 4600 50  0001 C CNN
@@
 $EndComp
 $Comp
-L GND #PWR027
+L GND #PWR028
 U 1 1 5AAF3C4B
 P 3000 4750
-F 0 "#PWR027" H 3000 4500 50  0001 C CNN
+F 0 "#PWR028" H 3000 4500 50  0001 C CNN
 F 1 "GND" H 3000 4600 50  0000 C CNN
 F 2 "" H 3000 4750 50  0001 C CNN
@@
 Connection ~ 4050 5050
 $Comp
-L GND #PWR028
+L GND #PWR029
 U 1 1 5AAF3C5F
 P 4050 5850
-F 0 "#PWR028" H 4050 5600 50  0001 C CNN
+F 0 "#PWR029" H 4050 5600 50  0001 C CNN
 F 1 "GND" H 4050 5700 50  0000 C CNN
 F 2 "" H 4050 5850 50  0001 C CNN
@@
 Connection ~ 4450 5050
 $Comp
-L GND #PWR029
+L GND #PWR030
 U 1 1 5AAF3C75
 P 4450 5850
-F 0 "#PWR029" H 4450 5600 50  0001 C CNN
+F 0 "#PWR030" H 4450 5600 50  0001 C CNN
 F 1 "GND" H 4450 5700 50  0000 C CNN
 F 2 "" H 4450 5850 50  0001 C CNN
@@
 F 3 "" H 6850 1900 50  0001 C CNN
 	1    6850 1900
-	0    1    1    0
+	0    -1   -1   0
 $EndComp
 Wire Wire Line
@@
 	6850 2050 6850 2650
 $Comp
-L GND #PWR030
+L GND #PWR031
 U 1 1 5AAF4525
 P 6850 3100
-F 0 "#PWR030" H 6850 2850 50  0001 C CNN
+F 0 "#PWR031" H 6850 2850 50  0001 C CNN
 F 1 "GND" H 6850 2950 50  0000 C CNN
 F 2 "" H 6850 3100 50  0001 C CNN
@@
 Connection ~ 6850 2400
 $Comp
-L GND #PWR031
+L GND #PWR032
 U 1 1 5AAF4536
 P 7300 3100
-F 0 "#PWR031" H 7300 2850 50  0001 C CNN
+F 0 "#PWR032" H 7300 2850 50  0001 C CNN
 F 1 "GND" H 7300 2950 50  0000 C CNN
 F 2 "" H 7300 3100 50  0001 C CNN
@@
 P 8850 1850
 F 0 "R35" V 8930 1850 50  0000 C CNN
-F 1 "1M" V 8750 1850 50  0000 C CNN
+F 1 "10K" V 8750 1850 50  0000 C CNN
 F 2 "Resistors_SMD:R_0805" V 8780 1850 50  0001 C CNN
 F 3 "" H 8850 1850 50  0001 C CNN
@@
 $EndComp
 $Comp
-L GND #PWR032
+L GND #PWR033
 U 1 1 5AAF454F
 P 8150 2000
-F 0 "#PWR032" H 8150 1750 50  0001 C CNN
+F 0 "#PWR033" H 8150 1750 50  0001 C CNN
 F 1 "GND" H 8150 1850 50  0000 C CNN
 F 2 "" H 8150 2000 50  0001 C CNN
@@
 Connection ~ 9200 2300
 $Comp
-L GND #PWR033
+L GND #PWR034
 U 1 1 5AAF4563
 P 9200 3100
-F 0 "#PWR033" H 9200 2850 50  0001 C CNN
+F 0 "#PWR034" H 9200 2850 50  0001 C CNN
 F 1 "GND" H 9200 2950 50  0000 C CNN
 F 2 "" H 9200 3100 50  0001 C CNN
@@
 Connection ~ 9600 2300
 $Comp
-L GND #PWR034
+L GND #PWR035
 U 1 1 5AAF4579
 P 9600 3100
-F 0 "#PWR034" H 9600 2850 50  0001 C CNN
+F 0 "#PWR035" H 9600 2850 50  0001 C CNN
 F 1 "GND" H 9600 2950 50  0000 C CNN
 F 2 "" H 9600 3100 50  0001 C CNN
@@
 F 3 "" H 6850 4650 50  0001 C CNN
 	1    6850 4650
-	0    1    1    0
+	0    -1   -1   0
 $EndComp
 Wire Wire Line
@@
 	6850 4800 6850 5400
 $Comp
-L GND #PWR035
+L GND #PWR036
 U 1 1 5AAF45D4
 P 6850 5850
-F 0 "#PWR035" H 6850 5600 50  0001 C CNN
+F 0 "#PWR036" H 6850 5600 50  0001 C CNN
 F 1 "GND" H 6850 5700 50  0000 C CNN
 F 2 "" H 6850 5850 50  0001 C CNN
@@
 Connection ~ 6850 5150
 $Comp
-L GND #PWR036
+L GND #PWR037
 U 1 1 5AAF45E5
 P 7300 5850
-F 0 "#PWR036" H 7300 5600 50  0001 C CNN
+F 0 "#PWR037" H 7300 5600 50  0001 C CNN
 F 1 "GND" H 7300 5700 50  0000 C CNN
 F 2 "" H 7300 5850 50  0001 C CNN
@@
 P 8850 4600
 F 0 "R36" V 8930 4600 50  0000 C CNN
-F 1 "1M" V 8750 4600 50  0000 C CNN
+F 1 "10K" V 8750 4600 50  0000 C CNN
 F 2 "Resistors_SMD:R_0805" V 8780 4600 50  0001 C CNN
 F 3 "" H 8850 4600 50  0001 C CNN
@@
 $EndComp
 $Comp
-L GND #PWR037
+L GND #PWR038
 U 1 1 5AAF45F2
 P 8150 4750
-F 0 "#PWR037" H 8150 4500 50  0001 C CNN
+F 0 "#PWR038" H 8150 4500 50  0001 C CNN
 F 1 "GND" H 8150 4600 50  0000 C CNN
 F 2 "" H 8150 4750 50  0001 C CNN
@@
 Connection ~ 9200 5050
 $Comp
-L GND #PWR038
+L GND #PWR039
 U 1 1 5AAF4606
 P 9200 5850
-F 0 "#PWR038" H 9200 5600 50  0001 C CNN
+F 0 "#PWR039" H 9200 5600 50  0001 C CNN
 F 1 "GND" H 9200 5700 50  0000 C CNN
 F 2 "" H 9200 5850 50  0001 C CNN
@@
 Connection ~ 9600 5050
 $Comp
-L GND #PWR039
+L GND #PWR040
 U 1 1 5AAF461C
 P 9600 5850
-F 0 "#PWR039" H 9600 5600 50  0001 C CNN
+F 0 "#PWR040" H 9600 5600 50  0001 C CNN
 F 1 "GND" H 9600 5700 50  0000 C CNN
 F 2 "" H 9600 5850 50  0001 C CNN
