File: FLAME_DETECT_5-8.sch (KiCad schematic (older format))
At the start: 58 parts, among them Q5 MMBT2907, Q6 MMBT2907, Q7 MMBT2907, Q8 MMBT2907, U3 LM358, U4 LM358

Commit message: - Finished footprints.
Parts:
- D15, D16, D17, D18, D21, D22, D23, D24: footprint Diodes_SMD:D_0805 -> Diodes_SMD:D_SOD-123
- D19, D20, D25, D26: footprint (none) -> LEDs:LED_1206
- FLAME_5, FLAME_6, FLAME_7, FLAME_8: footprint (none) -> flame-detect-pcb:KEYSTONE_SPADE_TERM_(1287)
- U3, U4: footprint (none) -> Housings_SOIC:SOIC-8_3.9x4.9mm_Pitch1.27mm
Changed lines of the file:
@@
 F 0 "FLAME_5" H 5050 1650 50  0000 C CNN
 F 1 "CONN_01X01" V 5150 1550 50  0001 C CNN
-F 2 "" H 5050 1550 50  0001 C CNN
+F 2 "flame-detect-pcb:KEYSTONE_SPADE_TERM_(1287)" H 5050 1550 50  0001 C CNN
 F 3 "" H 5050 1550 50  0001 C CNN
 	1    5050 1550
@@
 F 0 "D15" H 1800 2050 50  0000 C CNN
 F 1 "BAV21W-7-F" H 1800 1850 50  0000 C CNN
-F 2 "Diodes_SMD:D_0805" H 1800 1950 50  0001 C CNN
+F 2 "Diodes_SMD:D_SOD-123" H 1800 1950 50  0001 C CNN
 F 3 "" H 1800 1950 50  0001 C CNN
 	1    1800 1950
@@
 F 0 "U3" H 3600 2550 50  0000 L CNN
 F 1 "LM358" H 3600 2150 50  0000 L CNN
-F 2 "" H 3600 2350 50  0001 C CNN
+F 2 "Housings_SOIC:SOIC-8_3.9x4.9mm_Pitch1.27mm" H 3600 2350 50  0001 C CNN
 F 3 "" H 3600 2350 50  0001 C CNN
 	1    3600 2350
@@
 F 0 "D17" H 4150 2950 50  0000 C CNN
 F 1 "BZT52C5V1-TP" H 4150 2750 50  0000 C CNN
-F 2 "Diodes_SMD:D_0805" H 4150 2850 50  0001 C CNN
+F 2 "Diodes_SMD:D_SOD-123" H 4150 2850 50  0001 C CNN
 F 3 "" H 4150 2850 50  0001 C CNN
 	1    4150 2850
@@
 F 0 "D19" H 4550 3050 50  0000 C CNN
 F 1 "LED" H 4550 2850 50  0000 C CNN
-F 2 "" H 4550 2950 50  0001 C CNN
+F 2 "LEDs:LED_1206" H 4550 2950 50  0001 C CNN
 F 3 "" H 4550 2950 50  0001 C CNN
 	1    4550 2950
@@
 F 0 "FLAME_6" H 5050 4400 50  0000 C CNN
 F 1 "CONN_01X01" V 5150 4300 50  0001 C CNN
-F 2 "" H 5050 4300 50  0001 C CNN
+F 2 "flame-detect-pcb:KEYSTONE_SPADE_TERM_(1287)" H 5050 4300 50  0001 C CNN
 F 3 "" H 5050 4300 50  0001 C CNN
 	1    5050 4300
@@
 F 0 "D16" H 1800 4800 50  0000 C CNN
 F 1 "BAV21W-7-F" H 1800 4600 50  0000 C CNN
-F 2 "Diodes_SMD:D_0805" H 1800 4700 50  0001 C CNN
+F 2 "Diodes_SMD:D_SOD-123" H 1800 4700 50  0001 C CNN
 F 3 "" H 1800 4700 50  0001 C CNN
 	1    1800 4700
@@
 F 0 "D18" H 4150 5700 50  0000 C CNN
 F 1 "BZT52C5V1-TP" H 4150 5500 50  0000 C CNN
-F 2 "Diodes_SMD:D_0805" H 4150 5600 50  0001 C CNN
+F 2 "Diodes_SMD:D_SOD-123" H 4150 5600 50  0001 C CNN
 F 3 "" H 4150 5600 50  0001 C CNN
 	1    4150 5600
@@
 F 0 "D20" H 4550 5800 50  0000 C CNN
 F 1 "LED" H 4550 5600 50  0000 C CNN
-F 2 "" H 4550 5700 50  0001 C CNN
+F 2 "LEDs:LED_1206" H 4550 5700 50  0001 C CNN
 F 3 "" H 4550 5700 50  0001 C CNN
 	1    4550 5700
@@
 F 0 "FLAME_7" H 10200 1650 50  0000 C CNN
 F 1 "CONN_01X01" V 10300 1550 50  0001 C CNN
-F 2 "" H 10200 1550 50  0001 C CNN
+F 2 "flame-detect-pcb:KEYSTONE_SPADE_TERM_(1287)" H 10200 1550 50  0001 C CNN
 F 3 "" H 10200 1550 50  0001 C CNN
 	1    10200 1550
@@
 F 0 "D21" H 6950 2050 50  0000 C CNN
 F 1 "BAV21W-7-F" H 6950 1850 50  0000 C CNN
-F 2 "Diodes_SMD:D_0805" H 6950 1950 50  0001 C CNN
+F 2 "Diodes_SMD:D_SOD-123" H 6950 1950 50  0001 C CNN
 F 3 "" H 6950 1950 50  0001 C CNN
 	1    6950 1950
@@
 F 0 "U4" H 8750 2550 50  0000 L CNN
 F 1 "LM358" H 8750 2150 50  0000 L CNN
-F 2 "" H 8750 2350 50  0001 C CNN
+F 2 "Housings_SOIC:SOIC-8_3.9x4.9mm_Pitch1.27mm" H 8750 2350 50  0001 C CNN
 F 3 "" H 8750 2350 50  0001 C CNN
 	1    8750 2350
@@
 F 0 "D23" H 9300 2950 50  0000 C CNN
 F 1 "BZT52C5V1-TP" H 9300 2750 50  0000 C CNN
-F 2 "Diodes_SMD:D_0805" H 9300 2850 50  0001 C CNN
+F 2 "Diodes_SMD:D_SOD-123" H 9300 2850 50  0001 C CNN
 F 3 "" H 9300 2850 50  0001 C CNN
 	1    9300 2850
@@
 F 0 "D25" H 9700 3050 50  0000 C CNN
 F 1 "LED" H 9700 2850 50  0000 C CNN
-F 2 "" H 9700 2950 50  0001 C CNN
+F 2 "LEDs:LED_1206" H 9700 2950 50  0001 C CNN
 F 3 "" H 9700 2950 50  0001 C CNN
 	1    9700 2950
@@
 F 0 "FLAME_8" H 10200 4400 50  0000 C CNN
 F 1 "CONN_01X01" V 10300 4300 50  0001 C CNN
-F 2 "" H 10200 4300 50  0001 C CNN
+F 2 "flame-detect-pcb:KEYSTONE_SPADE_TERM_(1287)" H 10200 4300 50  0001 C CNN
 F 3 "" H 10200 4300 50  0001 C CNN
 	1    10200 4300
@@
 F 0 "D22" H 6950 4800 50  0000 C CNN
 F 1 "BAV21W-7-F" H 6950 4600 50  0000 C CNN
-F 2 "Diodes_SMD:D_0805" H 6950 4700 50  0001 C CNN
+F 2 "Diodes_SMD:D_SOD-123" H 6950 4700 50  0001 C CNN
 F 3 "" H 6950 4700 50  0001 C CNN
 	1    6950 4700
@@
 F 0 "D24" H 9300 5700 50  0000 C CNN
 F 1 "BZT52C5V1-TP" H 9300 5500 50  0000 C CNN
-F 2 "Diodes_SMD:D_0805" H 9300 5600 50  0001 C CNN
+F 2 "Diodes_SMD:D_SOD-123" H 9300 5600 50  0001 C CNN
 F 3 "" H 9300 5600 50  0001 C CNN
 	1    9300 5600
@@
 F 0 "D26" H 9700 5800 50  0000 C CNN
 F 1 "LED" H 9700 5600 50  0000 C CNN
-F 2 "" H 9700 5700 50  0001 C CNN
+F 2 "LEDs:LED_1206" H 9700 5700 50  0001 C CNN
 F 3 "" H 9700 5700 50  0001 C CNN
 	1    9700 5700
@@
 F 0 "U3" H 3600 5300 50  0000 L CNN
 F 1 "LM358" H 3600 4900 50  0000 L CNN
-F 2 "" H 3600 5100 50  0001 C CNN
+F 2 "Housings_SOIC:SOIC-8_3.9x4.9mm_Pitch1.27mm" H 3600 5100 50  0001 C CNN
 F 3 "" H 3600 5100 50  0001 C CNN
 	2    3600 5100
@@
 F 0 "U4" H 8750 5300 50  0000 L CNN
 F 1 "LM358" H 8750 4900 50  0000 L CNN
-F 2 "" H 8750 5100 50  0001 C CNN
+F 2 "Housings_SOIC:SOIC-8_3.9x4.9mm_Pitch1.27mm" H 8750 5100 50  0001 C CNN
 F 3 "" H 8750 5100 50  0001 C CNN
 	2    8750 5100

Commit message: - Fixed several bugs.
Parts:
- R49, R50, R63, R64: value 1M -> 10K
Connections:
- net at Q5.3 (C): now also D15.2 (A); no longer D15.1 (K)
- net at C20.1, R41.1, U3.3 (+): now also D15.1 (K); no longer D15.2 (A)
- net at Q6.3 (C): now also D16.2 (A); no longer D16.1 (K)
- net at C21.1, R42.1, U3.5 (+): now also D16.1 (K); no longer D16.2 (A)
- net at Q7.3 (C): now also D21.2 (A); no longer D21.1 (K)
- net at C24.1, R55.1, U4.3 (+): now also D21.1 (K); no longer D21.2 (A)
- net at Q8.3 (C): now also D22.2 (A); no longer D22.1 (K)
- net at C25.1, R56.1, U4.5 (+): now also D22.1 (K); no longer D22.2 (A)
Changed lines of the file:
@@
 F 3 "" H 1800 1950 50  0001 C CNN
 	1    1800 1950
-	0    1    1    0
+	0    -1   -1   0
 $EndComp
 Wire Wire Line
@@
 	1800 2100 1800 2700
 $Comp
-L GND #PWR040
+L GND #PWR041
 U 1 1 5AB012FC
 P 1800 3150
-F 0 "#PWR040" H 1800 2900 50  0001 C CNN
+F 0 "#PWR041" H 1800 2900 50  0001 C CNN
 F 1 "GND" H 1800 3000 50  0000 C CNN
 F 2 "" H 1800 3150 50  0001 C CNN
@@
 Connection ~ 1800 2450
 $Comp
-L GND #PWR041
+L GND #PWR042
 U 1 1 5AB0130E
 P 2250 3150
-F 0 "#PWR041" H 2250 2900 50  0001 C CNN
+F 0 "#PWR042" H 2250 2900 50  0001 C CNN
 F 1 "GND" H 2250 3000 50  0000 C CNN
 F 2 "" H 2250 3150 50  0001 C CNN
@@
 P 3800 1900
 F 0 "R49" V 3880 1900 50  0000 C CNN
-F 1 "1M" V 3700 1900 50  0000 C CNN
+F 1 "10K" V 3700 1900 50  0000 C CNN
 F 2 "Resistors_SMD:R_0805" V 3730 1900 50  0001 C CNN
 F 3 "" H 3800 1900 50  0001 C CNN
@@
 $EndComp
 $Comp
-L GND #PWR042
+L GND #PWR043
 U 1 1 5AB0132A
 P 3100 2050
-F 0 "#PWR042" H 3100 1800 50  0001 C CNN
+F 0 "#PWR043" H 3100 1800 50  0001 C CNN
 F 1 "GND" H 3100 1900 50  0000 C CNN
 F 2 "" H 3100 2050 50  0001 C CNN
@@
 Connection ~ 4150 2350
 $Comp
-L GND #PWR043
+L GND #PWR044
 U 1 1 5AB0133F
 P 4150 3150
-F 0 "#PWR043" H 4150 2900 50  0001 C CNN
+F 0 "#PWR044" H 4150 2900 50  0001 C CNN
 F 1 "GND" H 4150 3000 50  0000 C CNN
 F 2 "" H 4150 3150 50  0001 C CNN
@@
 Connection ~ 4550 2350
 $Comp
-L GND #PWR044
+L GND #PWR045
 U 1 1 5AB01357
 P 4550 3150
-F 0 "#PWR044" H 4550 2900 50  0001 C CNN
+F 0 "#PWR045" H 4550 2900 50  0001 C CNN
 F 1 "GND" H 4550 3000 50  0000 C CNN
 F 2 "" H 4550 3150 50  0001 C CNN
@@
 F 3 "" H 1800 4700 50  0001 C CNN
 	1    1800 4700
-	0    1    1    0
+	0    -1   -1   0
 $EndComp
 Wire Wire Line
@@
 	1800 4850 1800 5450
 $Comp
-L GND #PWR045
+L GND #PWR046
 U 1 1 5AB013BB
 P 1800 5900
-F 0 "#PWR045" H 1800 5650 50  0001 C CNN
+F 0 "#PWR046" H 1800 5650 50  0001 C CNN
 F 1 "GND" H 1800 5750 50  0000 C CNN
 F 2 "" H 1800 5900 50  0001 C CNN
@@
 Connection ~ 1800 5200
 $Comp
-L GND #PWR046
+L GND #PWR047
 U 1 1 5AB013CD
 P 2250 5900
-F 0 "#PWR046" H 2250 5650 50  0001 C CNN
+F 0 "#PWR047" H 2250 5650 50  0001 C CNN
 F 1 "GND" H 2250 5750 50  0000 C CNN
 F 2 "" H 2250 5900 50  0001 C CNN
@@
 P 3800 4650
 F 0 "R50" V 3880 4650 50  0000 C CNN
-F 1 "1M" V 3700 4650 50  0000 C CNN
+F 1 "10K" V 3700 4650 50  0000 C CNN
 F 2 "Resistors_SMD:R_0805" V 3730 4650 50  0001 C CNN
 F 3 "" H 3800 4650 50  0001 C CNN
@@
 $EndComp
 $Comp
-L GND #PWR047
+L GND #PWR048
 U 1 1 5AB013DB
 P 3100 4800
-F 0 "#PWR047" H 3100 4550 50  0001 C CNN
+F 0 "#PWR048" H 3100 4550 50  0001 C CNN
 F 1 "GND" H 3100 4650 50  0000 C CNN
 F 2 "" H 3100 4800 50  0001 C CNN
@@
 Connection ~ 4150 5100
 $Comp
-L GND #PWR048
+L GND #PWR049
 U 1 1 5AB013F0
 P 4150 5900
-F 0 "#PWR048" H 4150 5650 50  0001 C CNN
+F 0 "#PWR049" H 4150 5650 50  0001 C CNN
 F 1 "GND" H 4150 5750 50  0000 C CNN
 F 2 "" H 4150 5900 50  0001 C CNN
@@
 Connection ~ 4550 5100
 $Comp
-L GND #PWR049
+L GND #PWR050
 U 1 1 5AB01408
 P 4550 5900
-F 0 "#PWR049" H 4550 5650 50  0001 C CNN
+F 0 "#PWR050" H 4550 5650 50  0001 C CNN
 F 1 "GND" H 4550 5750 50  0000 C CNN
 F 2 "" H 4550 5900 50  0001 C CNN
@@
 F 3 "" H 6950 1950 50  0001 C CNN
 	1    6950 1950
-	0    1    1    0
+	0    -1   -1   0
 $EndComp
 Wire Wire Line
@@
 	6950 2100 6950 2700
 $Comp
-L GND #PWR050
+L GND #PWR051
 U 1 1 5AB0146C
 P 6950 3150
-F 0 "#PWR050" H 6950 2900 50  0001 C CNN
+F 0 "#PWR051" H 6950 2900 50  0001 C CNN
 F 1 "GND" H 6950 3000 50  0000 C CNN
 F 2 "" H 6950 3150 50  0001 C CNN
@@
 Connection ~ 6950 2450
 $Comp
-L GND #PWR051
+L GND #PWR052
 U 1 1 5AB0147E
 P 7400 3150
-F 0 "#PWR051" H 7400 2900 50  0001 C CNN
+F 0 "#PWR052" H 7400 2900 50  0001 C CNN
 F 1 "GND" H 7400 3000 50  0000 C CNN
 F 2 "" H 7400 3150 50  0001 C CNN
@@
 P 8950 1900
 F 0 "R63" V 9030 1900 50  0000 C CNN
-F 1 "1M" V 8850 1900 50  0000 C CNN
+F 1 "10K" V 8850 1900 50  0000 C CNN
 F 2 "Resistors_SMD:R_0805" V 8880 1900 50  0001 C CNN
 F 3 "" H 8950 1900 50  0001 C CNN
@@
 $EndComp
 $Comp
-L GND #PWR052
+L GND #PWR053
 U 1 1 5AB01493
 P 8250 2050
-F 0 "#PWR052" H 8250 1800 50  0001 C CNN
+F 0 "#PWR053" H 8250 1800 50  0001 C CNN
 F 1 "GND" H 8250 1900 50  0000 C CNN
 F 2 "" H 8250 2050 50  0001 C CNN
@@
 Connection ~ 9300 2350
 $Comp
-L GND #PWR053
+L GND #PWR054
 U 1 1 5AB014A8
 P 9300 3150
-F 0 "#PWR053" H 9300 2900 50  0001 C CNN
+F 0 "#PWR054" H 9300 2900 50  0001 C CNN
 F 1 "GND" H 9300 3000 50  0000 C CNN
 F 2 "" H 9300 3150 50  0001 C CNN
@@
 Connection ~ 9700 2350
 $Comp
-L GND #PWR054
+L GND #PWR055
 U 1 1 5AB014C0
 P 9700 3150
-F 0 "#PWR054" H 9700 2900 50  0001 C CNN
+F 0 "#PWR055" H 9700 2900 50  0001 C CNN
 F 1 "GND" H 9700 3000 50  0000 C CNN
 F 2 "" H 9700 3150 50  0001 C CNN
@@
 F 3 "" H 6950 4700 50  0001 C CNN
 	1    6950 4700
-	0    1    1    0
+	0    -1   -1   0
 $EndComp
 Wire Wire Line
@@
 	6950 4850 6950 5450
 $Comp
-L GND #PWR055
+L GND #PWR056
 U 1 1 5AB01524
 P 6950 5900
-F 0 "#PWR055" H 6950 5650 50  0001 C CNN
+F 0 "#PWR056" H 6950 5650 50  0001 C CNN
 F 1 "GND" H 6950 5750 50  0000 C CNN
 F 2 "" H 6950 5900 50  0001 C CNN
@@
 Connection ~ 6950 5200
 $Comp
-L GND #PWR056
+L GND #PWR057
 U 1 1 5AB01536
 P 7400 5900
-F 0 "#PWR056" H 7400 5650 50  0001 C CNN
+F 0 "#PWR057" H 7400 5650 50  0001 C CNN
 F 1 "GND" H 7400 5750 50  0000 C CNN
 F 2 "" H 7400 5900 50  0001 C CNN
@@
 P 8950 4650
 F 0 "R64" V 9030 4650 50  0000 C CNN
-F 1 "1M" V 8850 4650 50  0000 C CNN
+F 1 "10K" V 8850 4650 50  0000 C CNN
 F 2 "Resistors_SMD:R_0805" V 8880 4650 50  0001 C CNN
 F 3 "" H 8950 4650 50  0001 C CNN
@@
 $EndComp
 $Comp
-L GND #PWR057
+L GND #PWR058
 U 1 1 5AB01544
 P 8250 4800
-F 0 "#PWR057" H 8250 4550 50  0001 C CNN
+F 0 "#PWR058" H 8250 4550 50  0001 C CNN
 F 1 "GND" H 8250 4650 50  0000 C CNN
 F 2 "" H 8250 4800 50  0001 C CNN
@@
 Connection ~ 9300 5100
 $Comp
-L GND #PWR058
+L GND #PWR059
 U 1 1 5AB01559
 P 9300 5900
-F 0 "#PWR058" H 9300 5650 50  0001 C CNN
+F 0 "#PWR059" H 9300 5650 50  0001 C CNN
 F 1 "GND" H 9300 5750 50  0000 C CNN
 F 2 "" H 9300 5900 50  0001 C CNN
@@
 Connection ~ 9700 5100
 $Comp
-L GND #PWR059
+L GND #PWR060
 U 1 1 5AB01571
 P 9700 5900
-F 0 "#PWR059" H 9700 5650 50  0001 C CNN
+F 0 "#PWR060" H 9700 5650 50  0001 C CNN
 F 1 "GND" H 9700 5750 50  0000 C CNN
 F 2 "" H 9700 5900 50  0001 C CNN
